File: chaveador_mot_v2.1.kicad_sch (KiCad schematic)
At the start: 6 parts, among them Q1 IRF9540N, U1 4N25

Commit message: layout, primeiro save
Connections:
- net at Q1.1 (G), U1.5: now also R1.1; no longer R1.2
- net at D1.1 (K), Q1.3 (S): now also R1.2
Other:
- moved on the sheet: R1
Changed lines of the file:
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@@
 	(paper "A4")
+	(junction
+		(at 95.25 71.12)
+		(diameter 0)
+		(color 0 0 0 0)
+	)
 	(junction
 		(at 77.47 76.2)
@@
 		(diameter 0)
 		(color 0 0 0 0)
+	)
+	(wire
+		(pts
+			(xy 85.09 71.12) (xy 95.25 71.12)
+		)
+		(stroke
+			(width 0)
+			(type default)
+		)
 	)
 	(wire
@@
 	(symbol
 		(lib_id "Device:R")
-		(at 77.47 67.31 0)
+		(at 81.28 71.12 90)
 		(unit 1)
 		(body_style 1)
@@
 		(fields_autoplaced yes)
 		(property "Reference" "R1"
-			(at 80.01 66.0399 0)
-			(show_name no)
-			(do_not_autoplace no)
-			(effects
-				(font
-					(size 1.27 1.27)
-				)
-				(justify left)
+			(at 81.28 64.77 90)
+			(show_name no)
+			(do_not_autoplace no)
+			(effects
+				(font
+					(size 1.27 1.27)
+				)
 			)
 		)
 		(property "Value" "R"
-			(at 80.01 68.5799 0)
-			(show_name no)
-			(do_not_autoplace no)
-			(effects
-				(font
-					(size 1.27 1.27)
-				)
-				(justify left)
+			(at 81.28 67.31 90)
+			(show_name no)
+			(do_not_autoplace no)
+			(effects
+				(font
+					(size 1.27 1.27)
+				)
 			)
 		)
 		(property "Footprint" ""
-			(at 75.692 67.31 90)
+			(at 81.28 72.898 90)
 			(hide yes)
 			(show_name no)
@@
 		)
 		(property "Datasheet" ""
-			(at 77.47 67.31 0)
+			(at 81.28 71.12 0)
 			(hide yes)
 			(show_name no)
@@
 		)
 		(property "Description" "Resistor"
-			(at 77.47 67.31 0)
-			(hide yes)
-			(show_name no)
+			(at 81.28 71.12 0)
+			(hide yes)
+			(show_name no)
